Commit message: change all robot names

File: urdf/map_robot.xacro (robot description, xacro)
@@ -1,5 +1,5 @@
 <?xml version='1.0'?>
-<robot name="roborock" xmlns:xacro="http://www.ros.org/wiki/xacro">
-    <xacro:include filename="$(find roborock)/urdf/roborock.gazebo"/>
+<robot name="map_robot" xmlns:xacro="http://www.ros.org/wiki/xacro">
+    <xacro:include filename="$(find map_robot)/urdf/map_robot.gazebo"/>
     <material name="light_blue">
         <color rgba="0 170 255 1"/>
@@ -159,5 +159,5 @@
             <origin xyz="0.0 0 0" rpy=" 0 0 0"/>
             <geometry>
-                <mesh filename="package://roborock/meshes/hokuyo.dae"/>
+                <mesh filename="package://map_robot/meshes/hokuyo.dae"/>
             </geometry>
         </visual>

Commit message: change the footprint name

File: urdf/map_robot.xacro (robot description, xacro)
@@ -11,8 +11,8 @@
         <color rgba="255 255 204 1"/>
     </material>
-    <link name="robot_footprint"></link>
-    <joint name="robot_footprint_joint" type="fixed">
+    <link name="base_footprint"></link>
+    <joint name="base_footprint_joint" type="fixed">
         <origin xyz="0 0 0" rpy="0 0 0"/>
-        <parent link="robot_footprint"/>
+        <parent link="base_footprint"/>
         <child link="chassis"/>
     </joint>

Commit message: change the camera angle

File: urdf/map_robot.xacro (robot description, xacro)
@@ -140,5 +140,5 @@
     </link>
     <joint type="fixed" name="camera_joint">
-        <origin xyz="0.21 0 0" rpy="0 0 0"/>
+        <origin xyz="0.21 0 0" rpy="${-pi/2} 0 ${-pi/2}"/>
         <child link="camera"/>
         <parent link="chassis"/>

Commit message: wrong reference name in xacro?

File: urdf/map_robot.xacro (robot description, xacro)
@@ -120,5 +120,5 @@
         </visual>
     </link>
-    <link name='camera'>
+    <link name='camera_link'>
         <inertial>
             <mass value="0.1"/>

Commit message: need to change here too

File: urdf/map_robot.xacro (robot description, xacro)
@@ -141,5 +141,5 @@
     <joint type="fixed" name="camera_joint">
         <origin xyz="0.21 0 0" rpy="${-pi/2} 0 ${-pi/2}"/>
-        <child link="camera"/>
+        <child link="camera_link"/>
         <parent link="chassis"/>
     </joint>

Commit message: the image direction is wrong

File: urdf/map_robot.xacro (robot description, xacro)
@@ -140,5 +140,5 @@
     </link>
     <joint type="fixed" name="camera_joint">
-        <origin xyz="0.21 0 0" rpy="${-pi/2} 0 ${-pi/2}"/>
+        <origin xyz="0.21 0 0" rpy="0 0 ${-pi/2}"/>
         <child link="camera_link"/>
         <parent link="chassis"/>

Commit message: tweak directions

File: urdf/map_robot.xacro (robot description, xacro)
@@ -140,5 +140,5 @@
     </link>
     <joint type="fixed" name="camera_joint">
-        <origin xyz="0.21 0 0" rpy="0 0 ${-pi/2}"/>
+        <origin xyz="0.21 0 0" rpy="0 ${pi/2} ${pi/2}"/>
         <child link="camera_link"/>
         <parent link="chassis"/>

Commit message: tweak direction

File: urdf/map_robot.xacro (robot description, xacro)
@@ -140,5 +140,5 @@
     </link>
     <joint type="fixed" name="camera_joint">
-        <origin xyz="0.21 0 0" rpy="0 ${pi/2} ${pi/2}"/>
+        <origin xyz="0.21 0 0" rpy="0 ${pi/2} ${-pi/2}"/>
         <child link="camera_link"/>
         <parent link="chassis"/>

Commit message: tweak

File: urdf/map_robot.xacro (robot description, xacro)
@@ -140,5 +140,5 @@
     </link>
     <joint type="fixed" name="camera_joint">
-        <origin xyz="0.21 0 0" rpy="0 ${pi/2} ${-pi/2}"/>
+        <origin xyz="0.3 0 0" rpy="${-pi/2} 0 ${-pi/2}"/>
         <child link="camera_link"/>
         <parent link="chassis"/>

Commit message: change camera direction

File: urdf/map_robot.xacro (robot description, xacro)
@@ -123,9 +123,9 @@
         <inertial>
             <mass value="0.1"/>
-            <origin xyz="0.0 0 0" rpy=" 0 0 0"/>
+            <origin xyz="0.0 0 0" rpy="${pi/2} 0 0"/>
             <inertia ixx="1e-6" ixy="0" ixz="0" iyy="1e-6" iyz="0" izz="1e-6"/>
         </inertial>
         <collision name='camera_collision'>
-            <origin xyz="0.0 0 0" rpy=" 0 0 0"/>
+            <origin xyz="0.0 0 0" rpy="${pi/2} 0 0"/>
             <geometry>
                 <box size=".05 .05 .05"/>
@@ -133,5 +133,5 @@
         </collision>
         <visual name='camera_visual'>
-            <origin xyz="0.0 0 0" rpy=" 0 0 0"/>
+            <origin xyz="0.0 0 0" rpy="${pi/2} 0 0"/>
             <geometry>
                 <box size=".05 .05 .05"/>

Commit message: tweak

File: urdf/map_robot.xacro (robot description, xacro)
@@ -123,9 +123,9 @@
         <inertial>
             <mass value="0.1"/>
-            <origin xyz="0.0 0 0" rpy="${pi/2} 0 0"/>
+            <origin xyz="0.0 0 0" rpy="$0 0 0"/>
             <inertia ixx="1e-6" ixy="0" ixz="0" iyy="1e-6" iyz="0" izz="1e-6"/>
         </inertial>
         <collision name='camera_collision'>
-            <origin xyz="0.0 0 0" rpy="${pi/2} 0 0"/>
+            <origin xyz="0.0 0 0" rpy="$0 0 0"/>
             <geometry>
                 <box size=".05 .05 .05"/>
@@ -133,5 +133,5 @@
         </collision>
         <visual name='camera_visual'>
-            <origin xyz="0.0 0 0" rpy="${pi/2} 0 0"/>
+            <origin xyz="0.0 0 0" rpy="$0 0 0"/>
             <geometry>
                 <box size=".05 .05 .05"/>
@@ -140,5 +140,5 @@
     </link>
     <joint type="fixed" name="camera_joint">
-        <origin xyz="0.3 0 0" rpy="${-pi/2} 0 ${-pi/2}"/>
+        <origin xyz="0.3 0 0" rpy="$0 0 ${-pi/2}"/>
         <child link="camera_link"/>
         <parent link="chassis"/>

Commit message: typo

File: urdf/map_robot.xacro (robot description, xacro)
@@ -123,9 +123,9 @@
         <inertial>
             <mass value="0.1"/>
-            <origin xyz="0.0 0 0" rpy="$0 0 0"/>
+            <origin xyz="0.0 0 0" rpy="0 0 0"/>
             <inertia ixx="1e-6" ixy="0" ixz="0" iyy="1e-6" iyz="0" izz="1e-6"/>
         </inertial>
         <collision name='camera_collision'>
-            <origin xyz="0.0 0 0" rpy="$0 0 0"/>
+            <origin xyz="0.0 0 0" rpy="0 0 0"/>
             <geometry>
                 <box size=".05 .05 .05"/>
@@ -133,5 +133,5 @@
         </collision>
         <visual name='camera_visual'>
-            <origin xyz="0.0 0 0" rpy="$0 0 0"/>
+            <origin xyz="0.0 0 0" rpy="0 0 0"/>
             <geometry>
                 <box size=".05 .05 .05"/>
@@ -140,5 +140,5 @@
     </link>
     <joint type="fixed" name="camera_joint">
-        <origin xyz="0.3 0 0" rpy="$0 0 ${-pi/2}"/>
+        <origin xyz="0.3 0 0" rpy="0 0 ${-pi/2}"/>
         <child link="camera_link"/>
         <parent link="chassis"/>

Commit message: change axis

File: urdf/map_robot.xacro (robot description, xacro)
@@ -140,4 +140,5 @@
     </link>
     <joint type="fixed" name="camera_joint">
+        <axis xyz="0 1 0" />
         <origin xyz="0.3 0 0" rpy="0 0 ${-pi/2}"/>
         <child link="camera_link"/>

Commit message: change axis again

File: urdf/map_robot.xacro (robot description, xacro)
@@ -140,5 +140,5 @@
     </link>
     <joint type="fixed" name="camera_joint">
-        <axis xyz="0 1 0" />
+        <axis xyz="0 0 1" />
         <origin xyz="0.3 0 0" rpy="0 0 ${-pi/2}"/>
         <child link="camera_link"/>

Commit message: change again

File: urdf/map_robot.xacro (robot description, xacro)
@@ -140,5 +140,5 @@
     </link>
     <joint type="fixed" name="camera_joint">
-        <axis xyz="0 0 1" />
+        <axis xyz="1 0 0" />
         <origin xyz="0.3 0 0" rpy="0 0 ${-pi/2}"/>
         <child link="camera_link"/>

Commit message: change all back

File: urdf/map_robot.xacro (robot description, xacro)
@@ -140,6 +140,5 @@
     </link>
     <joint type="fixed" name="camera_joint">
-        <axis xyz="1 0 0" />
-        <origin xyz="0.3 0 0" rpy="0 0 ${-pi/2}"/>
+        <origin xyz="0.3 0 0" rpy="${-pi/2} 0 ${-pi/2}"/>
         <child link="camera_link"/>
         <parent link="chassis"/>

Commit message: tweak

File: urdf/map_robot.xacro (robot description, xacro)
@@ -140,5 +140,5 @@
     </link>
     <joint type="fixed" name="camera_joint">
-        <origin xyz="0.3 0 0" rpy="${-pi/2} 0 ${-pi/2}"/>
+        <origin xyz="0.3 0 0" rpy="${-pi/2} 0 ${-pi}"/>
         <child link="camera_link"/>
         <parent link="chassis"/>

Commit message: tweak

File: urdf/map_robot.xacro (robot description, xacro)
@@ -140,5 +140,5 @@
     </link>
     <joint type="fixed" name="camera_joint">
-        <origin xyz="0.3 0 0" rpy="${-pi/2} 0 ${-pi}"/>
+        <origin xyz="0.3 0 0" rpy="${-pi/2} ${-pi/2} ${-pi/2}"/>
         <child link="camera_link"/>
         <parent link="chassis"/>

Commit message: add an extra frame

File: urdf/map_robot.xacro (robot description, xacro)
@@ -140,8 +140,15 @@
     </link>
     <joint type="fixed" name="camera_joint">
-        <origin xyz="0.3 0 0" rpy="${-pi/2} ${-pi/2} ${-pi/2}"/>
+        <origin xyz="0.3 0 0" rpy="0 0 0"/>
         <child link="camera_link"/>
         <parent link="chassis"/>
     </joint>
+    <joint name="camera_optical_joint" type="fixed">
+        <!-- these values have to be these values otherwise the gazebo camera image won't be aligned properly with the frame it is supposedly originating from -->
+        <origin xyz="0 0 0" rpy="${-pi/2} 0 ${-pi/2}"/>
+        <parent link="camera_link"/>
+        <child link="camera_link_optical"/>
+    </joint>
+    <link name="camera_link_optical"></link>
     <link name='hokuyo'>
         <inertial>
